File: whirl.kicad_pcb (KiCad board)
At the start: 4 copper layers, 18.6 x 24.9 mm, 22 parts, among them J1 QWIIC, J2 Encoder, J3 TagConnect, J4 Power, J5 MOTOR, U1 STM32C011F4Ux, U2 STSPIN230

Commit message: rev:0x02
Connections:
- U1 pad 16: Net-(J3-SWDCLK) -> Net-(J3-SWDIO)
- U1 pad 17: Net-(J3-SWDIO) -> Net-(J3-SWDCLK)
Routing:
- net Net-(J3-SWDCLK): track 18.6 -> 17.2 mm
