File: whirl.kicad_sch (KiCad schematic)
At the start: 21 parts, among them J1 QWIIC, J2 Encoder, J3 TagConnect, J4 Power, J5 MOTOR, U1 STM32C011F4Ux, U2 STSPIN230

Commit message: rev:0x02
Connections:
- net at J3.2 (SWDIO): now also U1.16 (PA13); no longer U1.17 (PA14)
- net at J3.4 (SWDCLK): now also U1.17 (PA14); no longer U1.16 (PA13)
Changed lines of the file:
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@@
   (title_block
     (title "Whirl")
-    (date "2023-03-11")
-    (rev "0x01")
+    (date "2023-03-26")
+    (rev "0x02")
   )
   (junction (at 152.4 134.62) (diameter 0) (color 0 0 0 0)
@@
   (no_connect (at 123.19 119.38))
   (no_connect (at 133.35 119.38))
-  (wire (pts (xy 113.03 134.62) (xy 121.92 134.62))
-    (stroke (width 0) (type default))
-  )
   (wire (pts (xy 105.41 48.895) (xy 99.695 48.895))
     (stroke (width 0) (type default))
@@
     (stroke (width 0) (type default))
   )
+  (wire (pts (xy 115.57 133.35) (xy 115.57 134.62))
+    (stroke (width 0) (type default))
+  )
   (wire (pts (xy 111.76 184.15) (xy 111.76 188.595))
     (stroke (width 0) (type default))
@@
     (stroke (width 0) (type default))
   )
+  (wire (pts (xy 113.03 137.16) (xy 117.602 137.16))
+    (stroke (width 0) (type default))
+  )
+  (wire (pts (xy 119.38 133.35) (xy 115.57 133.35))
+    (stroke (width 0) (type default))
+  )
   (wire (pts (xy 129.54 199.39) (xy 133.985 199.39))
     (stroke (width 0) (type default))
@@
     (stroke (width 0) (type default))
   )
+  (wire (pts (xy 119.38 137.16) (xy 119.38 133.35))
+    (stroke (width 0) (type default))
+  )
   (wire (pts (xy 113.03 121.92) (xy 123.19 121.92))
     (stroke (width 0) (type default))
@@
     (stroke (width 0) (type default))
   )
+  (wire (pts (xy 117.602 137.16) (xy 117.602 134.62))
+    (stroke (width 0) (type default))
+  )
   (wire (pts (xy 96.52 188.595) (xy 102.87 188.595))
     (stroke (width 0) (type default))
@@
     (stroke (width 0) (type default))
   )
-  (wire (pts (xy 113.03 137.16) (xy 121.92 137.16))
-    (stroke (width 0) (type default))
-  )
   (wire (pts (xy 99.695 48.895) (xy 93.98 48.895))
     (stroke (width 0) (type default))
@@
     (stroke (width 0) (type default))
   )
+  (wire (pts (xy 117.602 134.62) (xy 121.92 134.62))
+    (stroke (width 0) (type default))
+  )
   (wire (pts (xy 88.9 219.71) (xy 94.615 219.71))
     (stroke (width 0) (type default))
@@
     (stroke (width 0) (type default))
   )
+  (wire (pts (xy 121.92 137.16) (xy 119.38 137.16))
+    (stroke (width 0) (type default))
+  )
   (wire (pts (xy 135.89 121.92) (xy 133.35 121.92))
     (stroke (width 0) (type default))
@@
     (stroke (width 0) (type default))
   )
+  (wire (pts (xy 115.57 134.62) (xy 113.03 134.62))
+    (stroke (width 0) (type default))
+  )
